File: badges/badges.kicad_pcb (KiCad board)
At the start: 2 copper layers, 99.5 x 55.1 mm, 18 parts, among them SW1 SW_Push, U1 LM555xN

Commit message: image + pcb
Parts:
- C1: moved to B.Cu
- moved R7 139.3 mm to (49.6, 157.6), turned to -75 degrees
- moved R6 138.6 mm to (49.0, 150.4), turned to 50 degrees
- moved R3 133.8 mm to (55.5, 141.1), turned to 70 degrees
- moved R8 132.8 mm to (66.4, 178.8), turned to -10 degrees
- moved R4 125.0 mm to (61.2, 136.2), turned to 10 degrees
- moved D1 118.5 mm to (53.0, 132.0), turned to 90 degrees
- moved R5 112.5 mm to (71.4, 132.0), turned to 20 degrees
- moved D2 103.9 mm to (65.2, 130.8), turned to 90 degrees
- moved R2 98.0 mm to (128.2, 166.1), turned to 90 degrees
- moved R1 93.1 mm to (128.2, 156.4), turned to 90 degrees
- moved D4 91.4 mm to (104.7, 176.5)
- moved D3 90.4 mm to (74.8, 126.0), turned to 90 degrees
- moved D5 75.2 mm to (119.8, 174.8)
- moved BT1 65.1 mm to (116.7, 150.6), turned to 90 degrees
- moved SW1 63.8 mm to (129.2, 175.1)
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Routing:
- net +6V: track 0.00 -> 162.3 mm
- net LED: track 0.00 -> 144.7 mm
- net Net-(D5-A): track 0.00 -> 77.2 mm
- net Net-(D6-A): track 0.00 -> 67.0 mm, vias 0 -> 1
- net Net-(D4-A): track 0.00 -> 66.6 mm
- net Net-(BT1-+): track 0.00 -> 48.0 mm
- net Net-(U1-THR): track 0.00 -> 29.8 mm
- net Net-(U1-DIS): track 0.00 -> 27.0 mm
- net Net-(D1-K): track 0.00 -> 5.94 mm
- net Net-(D2-K): track 0.00 -> 5.53 mm
- net Net-(D3-K): track 0.00 -> 5.11 mm
- added copper zone on B.Cu, net GND
- added copper zone on F.Cu, net GND
Other:
- board size 99.5 x 55.1 mm -> 98.3 x 63.4 mm
