File: badges/badges.kicad_pcb (KiCad board)
At the start: 2 copper layers, 98.3 x 63.4 mm, 18 parts, among them SW1 SW_Push, U1 LM555xN

Commit message: final hopefully
Connections:
- BT1 pad 2: Net-(BT1--) -> GND
