File: badges/badges.kicad_pcb (KiCad board)
At the start: 2 copper layers, 98.3 x 63.4 mm, 18 parts, among them SW1 SW_Push, U1 LM555xN

Commit message: UGH
Parts:
- moved BT1 19.7 mm to (135.4, 144.5), turned to 145 degrees
- moved U1 12.2 mm to (138.5, 150.6)
- moved C1 10.2 mm to (136.1, 163.2)
- moved D6 2.22 mm to (133.1, 170.0)
- moved R1 2.01 mm to (128.4, 158.4)
- moved R2 2.01 mm to (128.4, 168.1)
Routing:
- net Net-(BT1-+): track 48.0 -> 38.1 mm
- net Net-(U1-THR): track 29.8 -> 20.8 mm, vias 0 -> 1
- net +6V: track 162.3 -> 154.6 mm
- net Net-(U1-DIS): track 27.0 -> 19.3 mm
- net LED: track 144.7 -> 149.9 mm
- net Net-(D6-A): track 67.0 -> 67.6 mm
- net GND: vias 4 -> 0
