File: badges/badges.kicad_sch (KiCad schematic)
At the start: 18 parts, among them SW1 SW_Push, U1 LM555xN

Commit message: final hopefully
Connections:
- no-connect marks 0 -> 1
Changed lines of the file:
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@@
 		(color 0 0 0 0)
+	)
+	(no_connect
+		(at 119.38 92.71)
 	)
 	(wire
